Commit message: URDF file

File: gen3_2f85.urdf (robot description, URDF)
Before this commit: robot kinova, 19 links, 18 joints
Links:
- link base_link: geometry collision mesh filename=arms/gen3/7dof/meshes/base_link.dae; visual mesh filename=arms/gen3/7dof/meshes/base_link.dae
- link bracelet_link: geometry collision mesh filename=arms/gen3/7dof/meshes/bracelet_no_vision_link.dae; visual mesh filename=arms/gen3/7dof/meshes/bracelet_no_vision_link.dae
- link forearm_link: geometry collision mesh filename=arms/gen3/7dof/meshes/forearm_link.dae; visual mesh filename=arms/gen3/7dof/meshes/forearm_link.dae
- link half_arm_1_link: geometry collision mesh filename=arms/gen3/7dof/meshes/half_arm_1_link.dae; visual mesh filename=arms/gen3/7dof/meshes/half_arm_1_link.dae
- link half_arm_2_link: geometry collision mesh filename=arms/gen3/7dof/meshes/half_arm_2_link.dae; visual mesh filename=arms/gen3/7dof/meshes/half_arm_2_link.dae
- link robotiq_85_base_link: geometry collision mesh filename=robotiq_description/meshes/collision/2f_85/robotiq_base.stl; visual mesh filename=robotiq_description/meshes/visual/2f_85/robotiq_base.dae
- link robotiq_85_left_finger_link: geometry collision mesh filename=robotiq_description/meshes/collision/2f_85/left_finger.stl; visual mesh filename=robotiq_description/meshes/visual/2f_85/left_finger.dae
- link robotiq_85_left_finger_tip_link: geometry collision mesh filename=robotiq_description/meshes/collision/2f_85/left_finger_tip.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; visual mesh filename=robotiq_description/meshes/visual/2f_85/left_finger_tip.dae
- link robotiq_85_left_inner_knuckle_link: geometry collision mesh filename=robotiq_description/meshes/collision/2f_85/left_inner_knuck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; visual mesh filename=robotiq_description/meshes/visual/2f_85/left_inner_knuckle.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
- link robotiq_85_left_knuckle_link: geometry collision mesh filename=robotiq_description/meshes/collision/2f_85/left_knuckle.stl; visual mesh filename=robotiq_description/meshes/visual/2f_85/left_knuckle.dae
- link robotiq_85_right_finger_link: geometry collision mesh filename=robotiq_description/meshes/collision/2f_85/right_finger.stl; visual mesh filename=robotiq_description/meshes/visual/2f_85/right_finger.dae
- link robotiq_85_right_finger_tip_link: geometry collision mesh filename=robotiq_description/meshes/collision/2f_85/right_finger_tip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; visual mesh filename=robotiq_description/meshes/visual/2f_85/right_finger_tip.dae
- link robotiq_85_right_inner_knuckle_link: geometry collision mesh filename=robotiq_description/meshes/collision/2f_85/right_inner_knuc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; visual mesh filename=robotiq_description/meshes/visual/2f_85/right_inner_knuckle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
- link robotiq_85_right_knuckle_link: geometry collision mesh filename=robotiq_description/meshes/collision/2f_85/right_knuckle.stl; visual mesh filename=robotiq_description/meshes/visual/2f_85/right_knuckle.dae
- link shoulder_link: geometry collision mesh filename=arms/gen3/7dof/meshes/shoulder_link.dae; visual mesh filename=arms/gen3/7dof/meshes/shoulder_link.dae
- link spherical_wrist_1_link: geometry collision mesh filename=arms/gen3/7dof/meshes/spherical_wrist_1_link.dae; visual mesh filename=arms/gen3/7dof/meshes/spherical_wrist_1_link.dae
- link spherical_wrist_2_link: geometry collision mesh filename=arms/gen3/7dof/meshes/spherical_wrist_2_link.dae; visual mesh filename=arms/gen3/7dof/meshes/spherical_wrist_2_link.dae
Joints:
- removed joint joint_1
- removed joint joint_2
- removed joint joint_3
- removed joint joint_4
- removed joint joint_5
- removed joint joint_6
- removed joint joint_7
- added joint gen3_joint_1: type revolute, parent base_link, child shoulder_link, origin xyz=0 0 0.15643 rpy=3.1416 2.7629E-18 -4.9305E-36, axis 0 0 1, limit lower=-3.14159 upper=3.14159 effort=39 velocity=1.3963
- added joint gen3_joint_2: type revolute, parent shoulder_link, child half_arm_1_link, origin xyz=0 0.005375 -0.12838 rpy=1.5708 2.1343E-17 -1.1102E-16, axis 0 0 1, limit lower=-2.24 upper=2.24 effort=39 velocity=1.3963
- added joint gen3_joint_3: type revolute, parent half_arm_1_link, child half_arm_2_link, origin xyz=0 -0.21038 -0.006375 rpy=-1.5708 1.2326E-32 -2.9122E-16, axis 0 0 1, limit lower=-3.14159 upper=3.14159 effort=39 velocity=1.3963
- added joint gen3_joint_4: type revolute, parent half_arm_2_link, child forearm_link, origin xyz=0 0.006375 -0.21038 rpy=1.5708 -6.6954E-17 -1.6653E-16, axis 0 0 1, limit lower=-2.57 upper=2.57 effort=39 velocity=1.3963
- added joint gen3_joint_5: type revolute, parent forearm_link, child spherical_wrist_1_link, origin xyz=0 -0.20843 -0.006375 rpy=-1.5708 2.2204E-16 -6.373E-17, axis 0 0 1, limit lower=-3.14159 upper=3.14159 effort=9 velocity=1.2218
- added joint gen3_joint_6: type revolute, parent spherical_wrist_1_link, child spherical_wrist_2_link, origin xyz=0 0.00017505 -0.10593 rpy=1.5708 9.2076E-28 -8.2157E-15, axis 0 0 1, limit lower=-2.09 upper=2.09 effort=9 velocity=1.2218
- added joint gen3_joint_7: type revolute, parent spherical_wrist_2_link, child bracelet_link, origin xyz=0 -0.10593 -0.00017505 rpy=-1.5708 -5.5511E-17 9.6396E-17, axis 0 0 1, limit lower=-3.14159 upper=3.14159 effort=9 velocity=1.2218
- joint robotiq_85_left_finger_tip_joint: limit (none) -> lower=0.0 upper=0.8 effort=50 velocity=0.5; mimic joint=robotiq_85_left_knuckle_joint multiplier=-1 -> joint=robotiq_85_left_knuckle_joint multiplier=-1 offset=0; type continuous -> revolute
- joint robotiq_85_left_inner_knuckle_joint: limit (none) -> lower=0.0 upper=0.8 effort=50 velocity=0.5; mimic joint=robotiq_85_left_knuckle_joint -> joint=robotiq_85_left_knuckle_joint offset=0; type continuous -> revolute
- joint robotiq_85_right_finger_tip_joint: limit (none) -> lower=0.0 upper=0.8 effort=50 velocity=0.5; mimic joint=robotiq_85_left_knuckle_joint -> joint=robotiq_85_left_knuckle_joint offset=0; type continuous -> revolute
- joint robotiq_85_right_inner_knuckle_joint: limit (none) -> lower=0.0 upper=0.8 effort=50 velocity=0.5; mimic joint=robotiq_85_left_knuckle_joint multiplier=-1 -> joint=robotiq_85_left_knuckle_joint multiplier=-1 offset=0; type continuous -> revolute
- joint robotiq_85_right_knuckle_joint: mimic joint=robotiq_85_left_knuckle_joint multiplier=-1 -> joint=robotiq_85_left_knuckle_joint multiplier=-1 offset=0
