Commit message: last changes to effort limits

File: src/gen3/gen3lite_py/robot/gen3_lite.urdf (robot description, URDF)
Before this commit: robot gen3_lite, 15 links, 14 joints
Joints:
- joint joint_1: limit lower=-2.69 upper=2.69 effort=39 velocity=1.6 -> lower=-2.69 upper=2.69 effort=35 velocity=1.6
- joint joint_2: limit lower=-2.69 upper=2.69 effort=39 velocity=1.6 -> lower=-2.69 upper=2.69 effort=35 velocity=1.6
- joint joint_3: limit lower=-2.69 upper=2.69 effort=39 velocity=1.6 -> lower=-2.69 upper=2.69 effort=35 velocity=1.6
