Commit message: added twist integration to fake hardware

File: src/gen3/gen3_py/robot/gen3_2f85.urdf (robot description, URDF)
Before this commit: robot gen3_, 31 links, 30 joints
Links:
- added link gen3_tool_frame
Joints:
- added joint gen3_tool_frame_joint: type fixed, parent gen3_end_effector_link, child gen3_tool_frame, origin xyz=0 0 0.120 rpy=0 0 0.0, axis 0 0 0

File: src/gen3/gen3lite_py/robot/kortex.ros2_control.xacro (robot description, xacro)
@@ -32,20 +32,16 @@
         </xacro:if>
         <xacro:if value="${sim_isaac}">
-          <xacro:unless value="${moveit_active}">
-            <plugin>topic_based_ros2_control/TopicBasedSystem</plugin>
-            <param name="joint_commands_topic">${isaac_joint_commands}</param>
-            <param name="joint_states_topic">${isaac_joint_states}</param>
-          </xacro:unless>
+          <plugin>topic_based_ros2_control/TopicBasedSystem</plugin>
+          <param name="joint_commands_topic">${isaac_joint_commands}</param>
+          <param name="joint_states_topic">${isaac_joint_states}</param>
         </xacro:if>
         <xacro:if value="${use_fake_hardware}">
-          <xacro:unless value="${moveit_active}">
-            <plugin>mock_components/GenericSystem</plugin>
-            <param name="fake_sensor_commands">${fake_sensor_commands}</param>
-            <param name="state_following_offset">0.0</param>
-            <param name="calculate_dynamics">true</param>
-            <plugin>topic_based_ros2_control/TopicBasedSystem</plugin>
-            <param name="joint_commands_topic">/fake_joint_commands</param>
-            <param name="joint_states_topic">/fake_joint_states</param>
-          </xacro:unless>
+          <plugin>mock_components/GenericSystem</plugin>
+          <param name="fake_sensor_commands">${fake_sensor_commands}</param>
+          <param name="state_following_offset">0.0</param>
+          <param name="calculate_dynamics">true</param>
+          <plugin>topic_based_ros2_control/TopicBasedSystem</plugin>
+          <param name="joint_commands_topic">/fake_joint_commands</param>
+          <param name="joint_states_topic">/fake_joint_states</param>
         </xacro:if>
         <xacro:unless value="${use_fake_hardware or sim_gazebo or sim_isaac}">
